Commit message: Add inertia to links

File: urdf/test.urdf.xacro (robot description, xacro)
@@ -4,5 +4,6 @@
     <xacro:property name="M_PI" value="3.1415926535897931" />
     <!-- All variable xacro macros -->>
-    <xacro:property name="density" value="7874"/><<!-- iron -->>>
+    <!-- iron -->>
+    <xacro:property name="density" value="7874.0"/>
     <xacro:property name="body_w" value="0.40"/>
     <xacro:property name="body_d" value="0.30"/>
@@ -12,6 +13,6 @@
     <xacro:property name="leg_lower_r" value="0.02"/>
     <xacro:property name="leg_lower_l" value="0.25"/>
-    <xacro:property name="foot_l" value="0.15"/>
-    <xacro:property name="foot_w" value="0.25"/>
+    <xacro:property name="foot_w" value="0.15"/>
+    <xacro:property name="foot_d" value="0.25"/>
     <xacro:property name="foot_h" value="0.05"/>
     <xacro:property name="upper_leg_effort" value="6.5"/>
@@ -31,39 +32,39 @@
     <xacro:property name="joint_cylinder_mass" value="${
         density/(M_PI*joint_cylinder_r*joint_cylinder_r*joint_cylinder_l)
-    "/>
+    }"/>
     <xacro:property name="leg_lower_mass" value="${
-        density/(M_PI*leg_lower_r_r*leg_lower_r*leg_lower_l)
-    "/>
+        density/(M_PI*leg_lower_r*leg_lower_r*leg_lower_l)
+    }"/>
     <xacro:property name="leg_upper_mass" value="${
-        density/(M_PI*leg_upper_r_r*leg_upper_r*leg_upper_l)
-    "/>
+        density/(M_PI*leg_upper_r*leg_upper_r*leg_upper_l)
+    }"/>
     <xacro:property name="body_mass" value="${
-        density/(body_l*body_w*body_h)
-    "/>
+        density/(body_w*body_d*body_h)
+    }"/>
     <xacro:property name="foot_mass" value="${
-        density/(foot_l*foot_w*foot_h)
-    "/>
+        density/(foot_w*foot_d*foot_h)
+    }"/>
     <!-- inertial calculations -->>
-    <xacro:macro name="cylinder_inertial" params="name">
+    <xacro:macro name="cylinder_inertial" params="m r l">
         <inertial>
-            <mass value="${name}_mass"/>
+            <mass value="${m}"/>
             <inertia
-                ixx="${${name}_mass*(1/12*${name}_l**2 + 1/4*${name}_r**2)}",
-                ixy="0", ixy="0",
-                iyy="${${name}_mass*(1/12*${name}_l**2 + 1/4*${name}_r**2)}",
-                iyz="0",
-                izz="${0.5*${name}_mass*${name}_r**2)}"
+                ixx="${m*(1/12*l*l + 1/4*r*r)}"
+                ixy="0" ixz="0"
+                iyy="${m*(1/12*l*l + 1/4*r*r)}"
+                iyz="0"
+                izz="${1/2*m*r*r}"
             />
         </inertial>
     </xacro:macro>
-    <xacro:macro name="square_inertial" params="name">
+    <xacro:macro name="square_inertial" params="m w d h">
         <inertial>
-            <mass value="${name}_mass"/>
+            <mass value="${m}"/>
             <inertia
-                ixx="${1/12*${name}_mass*(${name}_h**2 + ${name}_d**2}",
-                ixy="0", ixz="0",
-                iyy="${1/12*${name}_mass*(${name}_w**2 + ${name}_d**2}",
-                iyz="0",
-                izz="${1/12*${name}_mass*(${name}_w**2 + ${name}_h**2}"
+                ixx="${1/12*m*(h*h + d*d)}"
+                ixy="0" ixz="0"
+                iyy="${1/12*m*(w*w + d*d)}"
+                iyz="0"
+                izz="${1/12*m*(w*w + h*h)}"
             />
         </inertial>
@@ -71,4 +72,5 @@
     <!-- All links and joints -->>
     <link name="body">
+        <xacro:square_inertial m="${body_mass}" w="${body_w}" d="${body_d}" h="${body_h}"/>
         <visual>
             <geometry>
@@ -80,4 +82,5 @@
     </link>
     <link name="left_leg_upper_joint_x">
+        <xacro:cylinder_inertial m="${joint_cylinder_mass}" r="${joint_cylinder_r}" l="${joint_cylinder_l}"/>
         <visual>
             <geometry>
@@ -89,4 +92,5 @@
     </link>
     <link name="right_leg_upper_joint_x">
+    <xacro:cylinder_inertial m="${joint_cylinder_mass}" r="${joint_cylinder_r}" l="${joint_cylinder_l}"/>
         <visual>
             <geometry>
@@ -112,4 +116,5 @@
     </joint>
     <link name="left_leg_upper_joint_y">
+        <xacro:cylinder_inertial m="${joint_cylinder_mass}" r="${joint_cylinder_r}" l="${joint_cylinder_l}"/>
         <visual>
             <geometry>
@@ -121,4 +126,5 @@
     </link>
     <link name="right_leg_upper_joint_y">
+        <xacro:cylinder_inertial m="${joint_cylinder_mass}" r="${joint_cylinder_r}" l="${joint_cylinder_l}"/>
         <visual>
             <geometry>
@@ -144,4 +150,5 @@
     </joint>
     <link name="left_leg_upper">
+        <xacro:cylinder_inertial m="${leg_upper_mass}" r="${leg_upper_r}" l="${leg_upper_l}"/>
         <visual>
             <geometry>
@@ -153,4 +160,5 @@
     </link>
     <link name="right_leg_upper">
+        <xacro:cylinder_inertial m="${leg_upper_mass}" r="${leg_upper_r}" l="${leg_upper_l}"/>
         <visual>
             <geometry>
@@ -172,4 +180,5 @@
     </joint>
     <link name="left_leg_knee_x">
+        <xacro:cylinder_inertial m="${joint_cylinder_mass}" r="${joint_cylinder_r}" l="${joint_cylinder_l}"/>
         <visual>
             <geometry>
@@ -181,4 +190,5 @@
     </link>
     <link name="right_leg_knee_x">
+        <xacro:cylinder_inertial m="${joint_cylinder_mass}" r="${joint_cylinder_r}" l="${joint_cylinder_l}"/>
         <visual>
             <geometry>
@@ -204,4 +214,5 @@
     </joint>
     <link name="left_leg_lower">
+        <xacro:cylinder_inertial m="${leg_lower_mass}" r="${leg_lower_r}" l="${leg_lower_l}"/>
         <visual>
             <geometry>
@@ -213,4 +224,5 @@
     </link>
     <link name="right_leg_lower">
+        <xacro:cylinder_inertial m="${leg_lower_mass}" r="${leg_lower_r}" l="${leg_lower_l}"/>
         <visual>
             <geometry>
@@ -232,4 +244,5 @@
     </joint>
     <link name="left_leg_lower_joint_x">
+        <xacro:cylinder_inertial m="${joint_cylinder_mass}" r="${joint_cylinder_r}" l="${joint_cylinder_l}"/>
         <visual>
             <geometry>
@@ -241,4 +254,5 @@
     </link>
     <link name="right_leg_lower_joint_x">
+        <xacro:cylinder_inertial m="${joint_cylinder_mass}" r="${joint_cylinder_r}" l="${joint_cylinder_l}"/>
         <visual>
             <geometry>
@@ -264,4 +278,5 @@
     </joint>
     <link name="left_leg_lower_joint_y">
+        <xacro:cylinder_inertial m="${joint_cylinder_mass}" r="${joint_cylinder_r}" l="${joint_cylinder_l}"/>
         <visual>
             <geometry>
@@ -273,4 +288,5 @@
     </link>
     <link name="right_leg_lower_joint_y">
+        <xacro:cylinder_inertial m="${joint_cylinder_mass}" r="${joint_cylinder_r}" l="${joint_cylinder_l}"/>
         <visual>
             <geometry>
@@ -296,19 +312,21 @@
     </joint>
     <link name="left_foot">
-        <visual>
-            <geometry>
-                <box size="${foot_l} ${foot_w} ${foot_h}"/>
-            </geometry>
-            <material name="red"/>
-            <origin xyz="0 -${foot_w/4} -${foot_h/2}"/>
+        <xacro:square_inertial m="${foot_mass}" w="${foot_w}" d="${foot_d}" h="${foot_h}"/>
+        <visual>
+            <geometry>
+                <box size="${foot_w} ${foot_d} ${foot_h}"/>
+            </geometry>
+            <material name="red"/>
+            <origin xyz="0 -${foot_d/4} -${foot_h/2}"/>
         </visual>
     </link>
     <link name="right_foot">
-        <visual>
-            <geometry>
-                <box size="${foot_l} ${foot_w} ${foot_h}"/>
-            </geometry>
-            <material name="red"/>
-            <origin xyz="0 -${foot_w/4} -${foot_h/2}"/>
+        <xacro:square_inertial m="${foot_mass}" w="${foot_w}" d="${foot_d}" h="${foot_h}"/>
+        <visual>
+            <geometry>
+                <box size="${foot_w} ${foot_d} ${foot_h}"/>
+            </geometry>
+            <material name="red"/>
+            <origin xyz="0 -${foot_d/4} -${foot_h/2}"/>
         </visual>
     </link>
