Commit message: Basic gazebo launch

File: urdf/biped.urdf.xacro (robot description, xacro)
@@ -71,4 +71,6 @@
     </xacro:macro>
     <!-- All links and joints -->>
+    <link name="base_link">
+    </link>
     <link name="body">
         <xacro:square_inertial m="${body_mass}" w="${body_w}" d="${body_d}" h="${body_h}"/>
@@ -80,5 +82,16 @@
             <material name="green"/>
         </visual>
-    </link>
+        <collision>
+            <geometry>
+                <box size="${body_w} ${body_d} ${body_h}"/>
+            </geometry>
+            <origin rpy="0 0 0" xyz="0 0 ${body_h/2}"/>
+        </collision>
+    </link>
+    <joint name="base_link_to_body" type="fixed">
+        <parent link="base_link"/>
+        <child link="body"/>
+        <origin xyz="0 0 0"/>
+    </joint>
     <link name="left_leg_upper_joint_x">
         <xacro:cylinder_inertial m="${joint_cylinder_mass}" r="${joint_cylinder_r}" l="${joint_cylinder_l}"/>
@@ -90,4 +103,10 @@
             <material name="yellow"/>
         </visual>
+        <collision>
+            <geometry>
+                <cylinder length="${joint_cylinder_l}" radius="${joint_cylinder_r}"/>
+            </geometry>
+            <origin xyz=" 0 0 -${joint_cylinder_r} " rpy="0 ${M_PI/2} 0"/>
+        </collision>
     </link>
     <link name="right_leg_upper_joint_x">
@@ -100,4 +119,10 @@
             <material name="yellow"/>
         </visual>
+        <collision>
+            <geometry>
+                <cylinder length="${joint_cylinder_l}" radius="${joint_cylinder_r}"/>
+            </geometry>
+            <origin xyz="0 0 -${joint_cylinder_r}" rpy="0 ${M_PI/2} 0"/>
+        </collision>
     </link>
     <joint name="body_to_left_leg_upper_joint_x" type="revolute">
@@ -124,4 +149,10 @@
             <material name="blue"/>
         </visual>
+        <collision>
+            <geometry>
+                <cylinder length="${joint_cylinder_l}" radius="${joint_cylinder_r}"/>
+            </geometry>
+            <origin xyz="0 0 -${joint_cylinder_r}" rpy="0 ${M_PI/2} ${M_PI/2}"/>
+        </collision>
     </link>
     <link name="right_leg_upper_joint_y">
@@ -134,4 +165,10 @@
             <material name="blue"/>
         </visual>
+        <collision>
+            <geometry>
+                <cylinder length="${joint_cylinder_l}" radius="${joint_cylinder_r}"/>
+            </geometry>
+            <origin xyz="0 0 -${joint_cylinder_r}" rpy="0 ${M_PI/2} ${M_PI/2}"/>
+        </collision>
     </link>
     <joint name="left_leg_upper_joint_x_to_left_leg_upper_joint_y" type="revolute">
@@ -158,4 +195,10 @@
             <material name="red"/>
         </visual>
+        <collision>
+            <geometry>
+                <cylinder length="${leg_upper_l}" radius="${leg_upper_r}"/>
+            </geometry>
+            <origin xyz="0 0 -${leg_upper_l/2}"/>
+        </collision>
     </link>
     <link name="right_leg_upper">
@@ -168,4 +211,10 @@
             <material name="red"/>
         </visual>
+        <collision>
+            <geometry>
+                <cylinder length="${leg_upper_l}" radius="${leg_upper_r}"/>
+            </geometry>
+            <origin xyz="0 0 -${leg_upper_l/2}"/>
+        </collision>
     </link>
     <joint name="left_leg_upper_joint_y_to_left_leg_upper" type="fixed">
@@ -188,4 +237,10 @@
             <material name="yellow"/>
         </visual>
+        <collision>
+            <geometry>
+                <cylinder length="${joint_cylinder_l}" radius="${joint_cylinder_r}"/>
+            </geometry>
+            <origin xyz="0 0 -${joint_cylinder_r}" rpy="0 ${M_PI/2} 0"/>
+        </collision>
     </link>
     <link name="right_leg_knee_x">
@@ -198,4 +253,10 @@
             <material name="yellow"/>
         </visual>
+        <collision>
+            <geometry>
+                <cylinder length="${joint_cylinder_l}" radius="${joint_cylinder_r}"/>
+            </geometry>
+            <origin xyz="0 0 -${joint_cylinder_r}" rpy="0 ${M_PI/2} 0"/>
+        </collision>
     </link>
     <joint name="left_leg_upper_to_left_leg_knee_x" type="revolute">
@@ -222,4 +283,10 @@
             <material name="red"/>
         </visual>
+        <collision>
+            <geometry>
+                <cylinder length="${leg_lower_l}" radius="${leg_lower_r}"/>
+            </geometry>
+            <origin xyz="0 0 -${leg_lower_l/2}"/>
+        </collision>
     </link>
     <link name="right_leg_lower">
@@ -232,4 +299,10 @@
             <material name="red"/>
         </visual>
+        <collision>
+            <geometry>
+                <cylinder length="${leg_lower_l}" radius="${leg_lower_r}"/>
+            </geometry>
+            <origin xyz="0 0 -${leg_lower_l/2}"/>
+        </collision>
     </link>
     <joint name="left_leg_knee_x_to_left_leg_lower" type="fixed">
@@ -252,4 +325,10 @@
             <material name="yellow"/>
         </visual>
+        <collision>
+            <geometry>
+                <cylinder length="${joint_cylinder_l}" radius="${joint_cylinder_r}"/>
+            </geometry>
+            <origin xyz=" 0 0 -${joint_cylinder_r} " rpy="0 ${M_PI/2} 0"/>
+        </collision>
     </link>
     <link name="right_leg_lower_joint_x">
@@ -262,4 +341,10 @@
             <material name="yellow"/>
         </visual>
+        <collision>
+            <geometry>
+                <cylinder length="${joint_cylinder_l}" radius="${joint_cylinder_r}"/>
+            </geometry>
+            <origin xyz=" 0 0 -${joint_cylinder_r} " rpy="0 ${M_PI/2} 0"/>
+        </collision>
     </link>
     <joint name="left_leg_lower_to_left_leg_lower_joint_x" type="revolute">
@@ -286,4 +371,10 @@
             <material name="blue"/>
         </visual>
+        <collision>
+            <geometry>
+                <cylinder length="${joint_cylinder_l}" radius="${joint_cylinder_r}"/>
+            </geometry>
+            <origin xyz=" 0 0 -${joint_cylinder_r} " rpy="0 ${M_PI/2} 0"/>
+        </collision>
     </link>
     <link name="right_leg_lower_joint_y">
@@ -296,4 +387,10 @@
             <material name="blue"/>
         </visual>
+        <collision>
+            <geometry>
+                <cylinder length="${joint_cylinder_l}" radius="${joint_cylinder_r}"/>
+            </geometry>
+            <origin xyz="0 0 -${joint_cylinder_r}" rpy="0 ${M_PI/2} ${M_PI/2}"/>
+        </collision>
     </link>
     <joint name="left_leg_lower_joint_x_to_left_leg_lower_joint_y" type="revolute">
@@ -317,7 +414,13 @@
                 <box size="${foot_w} ${foot_d} ${foot_h}"/>
             </geometry>
-            <material name="red"/>
             <origin xyz="0 -${foot_d/4} -${foot_h/2}"/>
-        </visual>
+            <material name="red"/>
+        </visual>
+        <collision>
+            <geometry>
+                <box size="${foot_w} ${foot_d} ${foot_h}"/>
+            </geometry>
+            <origin xyz="0 -${foot_d/4} -${foot_h/2}"/>
+        </collision>
     </link>
     <link name="right_foot">
@@ -327,7 +430,13 @@
                 <box size="${foot_w} ${foot_d} ${foot_h}"/>
             </geometry>
-            <material name="red"/>
             <origin xyz="0 -${foot_d/4} -${foot_h/2}"/>
-        </visual>
+            <material name="red"/>
+        </visual>
+        <collision>
+            <geometry>
+                <box size="${foot_w} ${foot_d} ${foot_h}"/>
+            </geometry>
+            <origin xyz="0 -${foot_d/4} -${foot_h/2}"/>
+        </collision>
     </link>
     <joint name="left_leg_lower_joint_y_to_left_foot" type="fixed">
@@ -341,3 +450,19 @@
         <origin xyz="0 0 -${joint_cylinder_r*2}"/>
     </joint>
+    <!-- Transmissions -->>
+    <transmission name="left_foot_pitch_trans">
+    <type>transmission_interface/SimpleTransmission</type>
+    <actuator name="$foot_pitch_motor">
+      <mechanicalReduction>1</mechanicalReduction>
+    </actuator>
+    <joint name="left_leg_lower_joint_x_to_left_leg_lower_joint_y">
+      <hardwareInterface>hardware_interface/PositionJointInterface</hardwareInterface>
+    </joint>
+  </transmission>
+    <!-- Gazebo plugin for ROS Control -->
+    <gazebo>
+        <plugin name="gazebo_ros_control" filename="libgazebo_ros_control.so">
+            <robotNamespace>/</robotNamespace>
+        </plugin>
+    </gazebo>
 </robot>
