Commit message: New xacro layout

File: urdf/inertials.urdf.xacro (robot description, xacro)
@@ -1,5 +1,5 @@
 <?xml version="1.0"?>
 <robot xmlns:xacro="http://www.ros.org/wiki/xacro">
-    <xacro:macro name="cylinder_inertial" params="rho r l">
+    <xacro:macro name="solid_cylinder_inertial" params="rho r l">
         <inertial>
             <mass value="${rho*(pi*r*r*l)}"/>
@@ -13,5 +13,5 @@
         </inertial>
     </xacro:macro>
-    <xacro:macro name="square_inertial" params="rho w d h">
+    <xacro:macro name="solid_cuboid_inertial" params="rho w d h">
         <inertial>
             <mass value="${rho*(w*d*h)}"/>

File: urdf/materials.urdf.xacro (robot description, xacro)
@@ -1,4 +1,4 @@
 <?xml version="1.0"?>
-<robot>
+<robot xmlns:xacro="http://www.ros.org/wiki/xacro">
     <material name="blue">
         <color rgba="${71/360} ${147/360} ${255/360} 1.0"/>
