Commit message: Properly spawn controllers

File: robot/biped.urdf.xacro (robot description, xacro)
@@ -11,5 +11,5 @@
     <gazebo>
         <plugin name="gazebo_ros_control" filename="libgazebo_ros_control.so">
-            <robotNamespace>/</robotNamespace>
+            <robotNamespace>/biped</robotNamespace>
         </plugin>
     </gazebo>

File: urdf/body.urdf.xacro (robot description, xacro)
@@ -11,4 +11,5 @@
         <origin xyz="0 0 ${body_h/2}"/>
     </xacro:default_fixed_joint>
+    <xacro:gazebo_ref prefix="body" material="Gazebo/Red"/>
     <!--======================================================-->>
 </robot>

File: urdf/common.urdf.xacro (robot description, xacro)
@@ -9,9 +9,12 @@
     <xacro:property name="leg_lower_r" value="0.02"/>
     <xacro:property name="leg_lower_l" value="0.25"/>
-    <xacro:property name="foot_w" value="0.15"/>
+    <xacro:property name="foot_w" value="0.25"/>
     <xacro:property name="foot_d" value="0.25"/>
     <xacro:property name="foot_h" value="0.05"/>
     <xacro:property name="default_effort" value="6.5"/>
     <xacro:property name="default_velocity" value="10"/>
+    <xacro:property name="default_damping" value="0.7"/>
+    <xacro:property name="default_mu1" value="0.1"/>
+    <xacro:property name="default_mu2" value="0.1"/>
     <xacro:property name="joint_cylinder_r" value="0.02"/>
     <xacro:property name="joint_cylinder_l" value="0.1"/>
@@ -57,5 +60,5 @@
     </xacro:macro>
     <xacro:macro name="default_rot_joint" params="parent child *origin *axis">
-        <joint name="${parent}_link_${child}_link_joint" type="revolute">
+        <joint name="${parent}_${child}_joint" type="revolute">
             <parent link="${parent}_link"/>
             <child link="${child}_link"/>
@@ -63,8 +66,9 @@
             <xacro:insert_block name="axis"/>
             <limit upper="${pi/2}" lower="-${pi/2}" effort="${default_effort}" velocity="${default_velocity}"/>
+            <dynamics damping="${default_damping}"/>
         </joint>
     </xacro:macro>
     <xacro:macro name="default_fixed_joint" params="parent child *origin">
-        <joint name="${parent}_link_${child}_link_joint" type="fixed">
+        <joint name="${parent}_${child}_joint" type="fixed">
             <parent link="${parent}_link"/>
             <child link="${child}_link"/>
@@ -74,12 +78,19 @@
     <xacro:macro name="joint_trans" params="parent child">
         <transmission name="${parent}_${child}_trans">
-            <type>transmission_interface/SimpleTransmission</type>
-            <actuator name="${parent}_link_${child}_link_joint_motor">
+            <type>EffortJointInterface</type>
+            <actuator name="${parent}_${child}_joint_motor">
                 <mechanicalReduction>1</mechanicalReduction>
             </actuator>
-            <joint name="${parent}_link_${child}_link_joint">
-                <hardwareInterface>hardware_interface/PositionJointInterface</hardwareInterface>
+            <joint name="${parent}_${child}_joint">
+                <hardwareInterface>hardware_interface/EffortJointInterface</hardwareInterface>
             </joint>
         </transmission>
     </xacro:macro>
+    <xacro:macro name="gazebo_ref" params="prefix material">
+        <gazebo reference="${prefix}_link">
+            <material>${material}</material>
+            <mu1>${default_mu1}</mu1>
+            <mu2>${default_mu2}</mu2>
+        </gazebo>
+    </xacro:macro>
 </robot>

File: urdf/feet.urdf.xacro (robot description, xacro)
@@ -11,4 +11,5 @@
     </xacro:default_rot_joint>
     <xacro:joint_trans parent="right_lower_leg" child="right_foot_roll"/>
+    <xacro:gazebo_ref prefix="right_foot_roll" material="Gazebo/Yellow"/>
     <!--======================================================-->>
     <!--======================================================-->>
@@ -22,4 +23,5 @@
     </xacro:default_rot_joint>
     <xacro:joint_trans parent="left_lower_leg" child="left_foot_roll"/>
+    <xacro:gazebo_ref prefix="left_foot_roll" material="Gazebo/Yellow"/>
     <!--======================================================-->>
     <!--======================================================-->>
@@ -33,4 +35,5 @@
     </xacro:default_rot_joint>
     <xacro:joint_trans parent="right_foot_roll" child="right_foot_pitch"/>
+    <xacro:gazebo_ref prefix="right_foot_pitch" material="Gazebo/Blue"/>
     <!--======================================================-->>
     <!--======================================================-->>
@@ -44,4 +47,5 @@
     </xacro:default_rot_joint>
     <xacro:joint_trans parent="left_foot_roll" child="left_foot_pitch"/>
+    <xacro:gazebo_ref prefix="left_foot_pitch" material="Gazebo/Blue"/>
     <!--======================================================-->>
     <!--======================================================-->>
@@ -52,4 +56,5 @@
         <origin xyz="0 0 -${joint_cylinder_r*2}"/>
     </xacro:default_fixed_joint>
+    <xacro:gazebo_ref prefix="right_foot" material="Gazebo/Red"/>
     <!--======================================================-->>
     <!--======================================================-->>
@@ -60,4 +65,5 @@
         <origin xyz="0 0 -${joint_cylinder_r*2}"/>
     </xacro:default_fixed_joint>
+    <xacro:gazebo_ref prefix="left_foot" material="Gazebo/Red"/>
     <!--======================================================-->>
 </robot>

File: urdf/lower_legs.urdf.xacro (robot description, xacro)
@@ -7,8 +7,9 @@
     </xacro:rot_link>
     <xacro:default_rot_joint parent="right_upper_leg" child="right_lower_leg_roll">
-        <origin xyz="0 0 -${leg_upper_l/2}"/>
+        <origin xyz="0 0 -${leg_upper_l/2+joint_cylinder_r}"/>
         <axis xyz="1 0 0"/>
     </xacro:default_rot_joint>
     <xacro:joint_trans parent="right_upper_leg" child="right_lower_leg_roll"/>
+    <xacro:gazebo_ref prefix="right_lower_leg_roll" material="Gazebo/Yellow"/>
     <!--======================================================-->>
     <!--======================================================-->>
@@ -18,8 +19,9 @@
     </xacro:rot_link>
     <xacro:default_rot_joint parent="left_upper_leg" child="left_lower_leg_roll">
-        <origin xyz="0 0 -${leg_upper_l/2}"/>
+        <origin xyz="0 0 -${leg_upper_l/2+joint_cylinder_r}"/>
         <axis xyz="1 0 0"/>
     </xacro:default_rot_joint>
     <xacro:joint_trans parent="left_upper_leg" child="left_lower_leg_roll"/>
+    <xacro:gazebo_ref prefix="left_lower_leg_roll" material="Gazebo/Yellow"/>
     <!--======================================================-->>
     <!--======================================================-->>
@@ -31,4 +33,5 @@
         <origin xyz="0 0 -${joint_cylinder_r+leg_lower_l/2}"/>
     </xacro:default_fixed_joint>
+    <xacro:gazebo_ref prefix="right_lower_leg" material="Gazebo/Red"/>
     <!--======================================================-->>
     <!--======================================================-->>
@@ -40,4 +43,5 @@
         <origin xyz="0 0 -${joint_cylinder_r+leg_lower_l/2}"/>
     </xacro:default_fixed_joint>
+    <xacro:gazebo_ref prefix="left_lower_leg" material="Gazebo/Red"/>
     <!--======================================================-->>
 </robot>

File: urdf/upper_legs.urdf.xacro (robot description, xacro)
@@ -11,4 +11,5 @@
     </xacro:default_rot_joint>
     <xacro:joint_trans parent="body" child="right_upper_leg_roll"/>
+    <xacro:gazebo_ref prefix="right_upper_leg_roll" material="Gazebo/Yellow"/>
     <!--======================================================-->>
     <!--======================================================-->>
@@ -22,4 +23,5 @@
     </xacro:default_rot_joint>
     <xacro:joint_trans parent="body" child="left_upper_leg_roll"/>
+    <xacro:gazebo_ref prefix="left_upper_leg_roll" material="Gazebo/Yellow"/>
     <!--======================================================-->>
     <!--======================================================-->>
@@ -33,4 +35,5 @@
     </xacro:default_rot_joint>
     <xacro:joint_trans parent="right_upper_leg_roll" child="right_upper_leg_pitch"/>
+    <xacro:gazebo_ref prefix="right_upper_leg_pitch" material="Gazebo/Blue"/>
     <!--======================================================-->>
     <!--======================================================-->>
@@ -44,4 +47,5 @@
     </xacro:default_rot_joint>
     <xacro:joint_trans parent="left_upper_leg_roll" child="left_upper_leg_pitch"/>
+    <xacro:gazebo_ref prefix="left_upper_leg_pitch" material="Gazebo/Blue"/>
     <!--======================================================-->>
     <!--======================================================-->>
@@ -53,4 +57,5 @@
         <origin xyz="0 0 -${joint_cylinder_r+leg_upper_l/2}"/>
     </xacro:default_fixed_joint>
+    <xacro:gazebo_ref prefix="right_upper_leg" material="Gazebo/Red"/>
     <!--======================================================-->>
     <!--======================================================-->>
@@ -62,4 +67,5 @@
         <origin xyz="0 0 -${joint_cylinder_r+leg_upper_l/2}"/>
     </xacro:default_fixed_joint>
+    <xacro:gazebo_ref prefix="left_upper_leg" material="Gazebo/Red"/>
     <!--======================================================-->>
 </robot>

Commit message: Refine layout

File: robot/biped.urdf.xacro (robot description, xacro)
@@ -4,8 +4,26 @@
     <xacro:include filename="$(find biped_description)/urdf/inertials.urdf.xacro"/>
     <xacro:include filename="$(find biped_description)/urdf/materials.urdf.xacro"/>
-    <xacro:include filename="$(find biped_description)/urdf/body.urdf.xacro"/>
-    <xacro:include filename="$(find biped_description)/urdf/upper_legs.urdf.xacro"/>
-    <xacro:include filename="$(find biped_description)/urdf/lower_legs.urdf.xacro"/>
-    <xacro:include filename="$(find biped_description)/urdf/feet.urdf.xacro"/>
+    <xacro:include filename="$(find biped_description)/urdf/macros.urdf.xacro"/>
+    <xacro:property name="body_w" value="0.40"/>
+    <xacro:property name="body_d" value="0.30"/>
+    <xacro:property name="body_h" value="0.60"/>
+    <xacro:property name="leg_upper_r" value="0.04"/>
+    <xacro:property name="leg_upper_l" value="0.20"/>
+    <xacro:property name="leg_lower_r" value="0.02"/>
+    <xacro:property name="leg_lower_l" value="0.25"/>
+    <xacro:property name="foot_w" value="0.15"/>
+    <xacro:property name="foot_d" value="0.20"/>
+    <xacro:property name="foot_h" value="0.05"/>
+    <xacro:property name="default_effort" value="1000"/>
+    <xacro:property name="default_velocity" value="50"/>
+    <xacro:property name="default_damping" value="0.7"/>
+    <xacro:property name="default_mu1" value="100"/>
+    <xacro:property name="default_mu2" value="100"/>
+    <xacro:property name="joint_cylinder_r" value="0.02"/>
+    <xacro:property name="joint_cylinder_l" value="0.1"/>
+    <xacro:include filename="$(find biped_description)/urdf/biped/body.urdf.xacro"/>
+    <xacro:include filename="$(find biped_description)/urdf/biped/upper_legs.urdf.xacro"/>
+    <xacro:include filename="$(find biped_description)/urdf/biped/lower_legs.urdf.xacro"/>
+    <xacro:include filename="$(find biped_description)/urdf/biped/feet.urdf.xacro"/>
     <!-- Gazebo plugin for ROS Control -->
     <gazebo>

File: urdf/biped/feet.urdf.xacro (robot description, xacro)
@@ -7,5 +7,5 @@
     </xacro:rot_link>
     <xacro:default_rot_joint parent="right_lower_leg" child="right_foot_roll">
-        <origin xyz="0 0 -${leg_lower_l/2}"/>
+        <origin xyz="0 0 -${leg_lower_l/2+joint_cylinder_r}"/>
         <axis xyz="1 0 0"/>
     </xacro:default_rot_joint>
@@ -19,5 +19,5 @@
     </xacro:rot_link>
     <xacro:default_rot_joint parent="left_lower_leg" child="left_foot_roll">
-        <origin xyz="0 0 -${leg_lower_l/2}"/>
+        <origin xyz="0 0 -${leg_lower_l/2+joint_cylinder_r}"/>
         <axis xyz="1 0 0"/>
     </xacro:default_rot_joint>
@@ -54,5 +54,5 @@
     </xacro:cuboid_link>
     <xacro:default_fixed_joint parent="right_foot_pitch" child="right_foot">
-        <origin xyz="0 0 -${joint_cylinder_r*2}"/>
+        <origin xyz="0 0 -${joint_cylinder_r+foot_h/2}"/>
     </xacro:default_fixed_joint>
     <xacro:gazebo_ref prefix="right_foot" material="Gazebo/Red"/>
@@ -63,5 +63,5 @@
     </xacro:cuboid_link>
     <xacro:default_fixed_joint parent="left_foot_pitch" child="left_foot">
-        <origin xyz="0 0 -${joint_cylinder_r*2}"/>
+        <origin xyz="0 0 -${joint_cylinder_r+foot_h/2}"/>
     </xacro:default_fixed_joint>
     <xacro:gazebo_ref prefix="left_foot" material="Gazebo/Red"/>

File: urdf/common.urdf.xacro (robot description, xacro)
@@ -1,96 +1,5 @@
 <?xml version="1.0"?>
 <robot xmlns:xacro="http://www.ros.org/wiki/xacro">
-    <xacro:property name="rho_Fe" value="7874.0"/>
-    <xacro:property name="body_w" value="0.40"/>
-    <xacro:property name="body_d" value="0.30"/>
-    <xacro:property name="body_h" value="0.60"/>
-    <xacro:property name="leg_upper_r" value="0.04"/>
-    <xacro:property name="leg_upper_l" value="0.20"/>
-    <xacro:property name="leg_lower_r" value="0.02"/>
-    <xacro:property name="leg_lower_l" value="0.25"/>
-    <xacro:property name="foot_w" value="0.25"/>
-    <xacro:property name="foot_d" value="0.25"/>
-    <xacro:property name="foot_h" value="0.05"/>
-    <xacro:property name="default_effort" value="6.5"/>
-    <xacro:property name="default_velocity" value="10"/>
-    <xacro:property name="default_damping" value="0.7"/>
-    <xacro:property name="default_mu1" value="0.1"/>
-    <xacro:property name="default_mu2" value="0.1"/>
-    <xacro:property name="joint_cylinder_r" value="0.02"/>
-    <xacro:property name="joint_cylinder_l" value="0.1"/>
-    <xacro:macro name="rot_link" params="prefix rho r l *rot_origin *material">
-        <link name="${prefix}_link">
-            <xacro:solid_cylinder_inertial rho="${rho}" r="${r}" l="${l}"/>
-            <visual>
-                <geometry>
-                    <cylinder length="${l}" radius="${r}"/>
-                </geometry>
-                <xacro:insert_block name="rot_origin"/>
-                <xacro:insert_block name="material"/>
-            </visual>
-            <collision>
-                <geometry>
-                    <cylinder length="${l}" radius="${r}"/>
-                </geometry>
-                <xacro:insert_block name="rot_origin"/>
-            </collision>
-        </link>
-    </xacro:macro>
-    <xacro:macro name="rot_x_origin">
-        <origin rpy="0 ${pi/2} 0"/>
-    </xacro:macro>
-    <xacro:macro name="rot_y_origin">
-        <origin rpy="0 ${pi/2} ${pi/2}"/>
-    </xacro:macro>
-    <xacro:macro name="cuboid_link" params="prefix rho w d h *material">
-        <link name="${prefix}_link">
-            <xacro:solid_cuboid_inertial rho="${rho}" w="${w}" d="${d}" h="${h}"/>
-            <visual>
-                <geometry>
-                    <box size="${w} ${d} ${h}"/>
-                </geometry>
-                <xacro:insert_block name="material"/>
-            </visual>
-            <collision>
-                <geometry>
-                    <box size="${w} ${d} ${h}"/>
-                </geometry>
-            </collision>
-        </link>
-    </xacro:macro>
-    <xacro:macro name="default_rot_joint" params="parent child *origin *axis">
-        <joint name="${parent}_${child}_joint" type="revolute">
-            <parent link="${parent}_link"/>
-            <child link="${child}_link"/>
-            <xacro:insert_block name="origin"/>
-            <xacro:insert_block name="axis"/>
-            <limit upper="${pi/2}" lower="-${pi/2}" effort="${default_effort}" velocity="${default_velocity}"/>
-            <dynamics damping="${default_damping}"/>
-        </joint>
-    </xacro:macro>
-    <xacro:macro name="default_fixed_joint" params="parent child *origin">
-        <joint name="${parent}_${child}_joint" type="fixed">
-            <parent link="${parent}_link"/>
-            <child link="${child}_link"/>
-            <xacro:insert_block name="origin"/>
-        </joint>
-    </xacro:macro>
-    <xacro:macro name="joint_trans" params="parent child">
-        <transmission name="${parent}_${child}_trans">
-            <type>EffortJointInterface</type>
-            <actuator name="${parent}_${child}_joint_motor">
-                <mechanicalReduction>1</mechanicalReduction>
-            </actuator>
-            <joint name="${parent}_${child}_joint">
-                <hardwareInterface>hardware_interface/EffortJointInterface</hardwareInterface>
-            </joint>
-        </transmission>
-    </xacro:macro>
-    <xacro:macro name="gazebo_ref" params="prefix material">
-        <gazebo reference="${prefix}_link">
-            <material>${material}</material>
-            <mu1>${default_mu1}</mu1>
-            <mu2>${default_mu2}</mu2>
-        </gazebo>
-    </xacro:macro>
+    <xacro:property name="rho_Fe" value="7874"/>
+    <xacro:property name="rho_PLA" value="1024"/>
 </robot>
