Commit message: Splitting common macros to seperate package

File: robot/biped.urdf.xacro (robot description, xacro)
@@ -1,8 +1,16 @@
 <?xml version="1.0"?>
 <robot xmlns:xacro="http://www.ros.org/wiki/xacro" name="biped">
-    <xacro:include filename="$(find biped_description)/urdf/common.urdf.xacro"/>
-    <xacro:include filename="$(find biped_description)/urdf/inertials.urdf.xacro"/>
-    <xacro:include filename="$(find biped_description)/urdf/materials.urdf.xacro"/>
-    <xacro:include filename="$(find biped_description)/urdf/macros.urdf.xacro"/>
+    <xacro:include filename="$(find xacro_common)/common.urdf.xacro"/>
+    <xacro:include filename="$(find xacro_common)/constants.urdf.xacro"/>
+    <xacro:include filename="$(find xacro_common)/gazebo.urdf.xacro"/>
+    <xacro:include filename="$(find xacro_common)/links.urdf.xacro"/>
+    <xacro:include filename="$(find xacro_common)/joints.urdf.xacro"/>
+    <xacro:include filename="$(find xacro_common)/inertials.urdf.xacro"/>
+    <xacro:include filename="$(find xacro_common)/materials.urdf.xacro"/>
+    <xacro:include filename="$(find xacro_common)/transmissions.urdf.xacro"/>
+    <xacro:include filename="$(find biped_description)/urdf/biped/body.urdf.xacro"/>
+    <xacro:include filename="$(find biped_description)/urdf/biped/upper_legs.urdf.xacro"/>
+    <xacro:include filename="$(find biped_description)/urdf/biped/lower_legs.urdf.xacro"/>
+    <xacro:include filename="$(find biped_description)/urdf/biped/feet.urdf.xacro"/>
     <xacro:property name="body_w" value="0.40"/>
     <xacro:property name="body_d" value="0.30"/>
@@ -15,15 +23,20 @@
     <xacro:property name="foot_d" value="0.20"/>
     <xacro:property name="foot_h" value="0.05"/>
-    <xacro:property name="default_effort" value="1000"/>
-    <xacro:property name="default_velocity" value="50"/>
-    <xacro:property name="default_damping" value="0.7"/>
-    <xacro:property name="default_mu1" value="100"/>
-    <xacro:property name="default_mu2" value="100"/>
+    <xacro:property name="effort" value="1000"/>
+    <xacro:property name="velocity" value="50"/>
+    <xacro:property name="damping" value="0.7"/>
+    <xacro:property name="mu1" value="100"/>
+    <xacro:property name="mu2" value="100"/>
     <xacro:property name="joint_cylinder_r" value="0.02"/>
     <xacro:property name="joint_cylinder_l" value="0.1"/>
-    <xacro:include filename="$(find biped_description)/urdf/biped/body.urdf.xacro"/>
-    <xacro:include filename="$(find biped_description)/urdf/biped/upper_legs.urdf.xacro"/>
-    <xacro:include filename="$(find biped_description)/urdf/biped/lower_legs.urdf.xacro"/>
-    <xacro:include filename="$(find biped_description)/urdf/biped/feet.urdf.xacro"/>
+    <!-- Place parts-->>
+    <xacro:base/>
+    <xacro:body name="body" parent="base"/>
+    <xacro:upper_leg name="right_upper_leg" parent="body" reflect="1"/>
+    <xacro:upper_leg name="left_upper_leg" parent="body" reflect="-1"/>
+    <xacro:lower_leg name="right_lower_leg" parent="right_upper_leg"/>
+    <xacro:lower_leg name="left_lower_leg" parent="left_upper_leg"/>
+    <xacro:foot name="right_foot" parent="right_lower_leg"/>
+    <xacro:foot name="left_foot" parent="left_lower_leg"/>
     <!-- Gazebo plugin for ROS Control -->
     <gazebo>

File: urdf/biped/body.urdf.xacro (robot description, xacro)
@@ -1,15 +1,12 @@
 <?xml version="1.0"?>
 <robot xmlns:xacro="http://www.ros.org/wiki/xacro">
-    <!--======================================================-->>
-    <link name="base_link">
-    </link>
-    <!--======================================================-->>
-    <xacro:cuboid_link prefix="body" rho="${rho_Fe}" w="${body_w}" d="${body_d}" h="${body_h}">
-        <material name="red"/>
-    </xacro:cuboid_link>
-    <xacro:default_fixed_joint parent="base" child="body">
-        <origin xyz="0 0 ${body_h/2}"/>
-    </xacro:default_fixed_joint>
-    <xacro:gazebo_ref prefix="body" material="Gazebo/Red"/>
-    <!--======================================================-->>
+    <xacro:macro name="body" params="name parent">
+        <xacro:solid_cuboid_link prefix="${name}" rho="${rho_Fe}" w="${body_w}" d="${body_d}" h="${body_h}">
+            <material name="red"/>
+        </xacro:solid_cuboid_link>
+        <xacro:fixed_joint parent="${parent}" child="${name}">
+            <origin xyz="0 0 ${body_h/2}"/>
+        </xacro:fixed_joint>
+        <xacro:gaz_link prefix="${name}" material="Gazebo/Red" mu1="${mu1}" mu2="${mu2}"/>
+    </xacro:macro>
 </robot>

File: urdf/biped/feet.urdf.xacro (robot description, xacro)
@@ -1,69 +1,34 @@
 <?xml version="1.0"?>
 <robot xmlns:xacro="http://www.ros.org/wiki/xacro">
-    <!--======================================================-->>
-    <xacro:rot_link prefix="right_foot_roll" rho="${rho_Fe}" r="${joint_cylinder_r}" l="${joint_cylinder_l}">
-        <xacro:rot_x_origin/>
-        <material name="yellow"/>
-    </xacro:rot_link>
-    <xacro:default_rot_joint parent="right_lower_leg" child="right_foot_roll">
-        <origin xyz="0 0 -${leg_lower_l/2+joint_cylinder_r}"/>
-        <axis xyz="1 0 0"/>
-    </xacro:default_rot_joint>
-    <xacro:joint_trans parent="right_lower_leg" child="right_foot_roll"/>
-    <xacro:gazebo_ref prefix="right_foot_roll" material="Gazebo/Yellow"/>
-    <!--======================================================-->>
-    <!--======================================================-->>
-    <xacro:rot_link prefix="left_foot_roll" rho="${rho_Fe}" r="${joint_cylinder_r}" l="${joint_cylinder_l}">
-        <xacro:rot_x_origin/>
-        <material name="yellow"/>
-    </xacro:rot_link>
-    <xacro:default_rot_joint parent="left_lower_leg" child="left_foot_roll">
-        <origin xyz="0 0 -${leg_lower_l/2+joint_cylinder_r}"/>
-        <axis xyz="1 0 0"/>
-    </xacro:default_rot_joint>
-    <xacro:joint_trans parent="left_lower_leg" child="left_foot_roll"/>
-    <xacro:gazebo_ref prefix="left_foot_roll" material="Gazebo/Yellow"/>
-    <!--======================================================-->>
-    <!--======================================================-->>
-    <xacro:rot_link prefix="right_foot_pitch" rho="${rho_Fe}" r="${joint_cylinder_r}" l="${joint_cylinder_l}">
-        <xacro:rot_y_origin/>
-        <material name="blue"/>
-    </xacro:rot_link>
-    <xacro:default_rot_joint parent="right_foot_roll" child="right_foot_pitch">
-        <origin xyz="0 0 ${-2*joint_cylinder_r}"/>
-        <axis xyz="0 1 0"/>
-    </xacro:default_rot_joint>
-    <xacro:joint_trans parent="right_foot_roll" child="right_foot_pitch"/>
-    <xacro:gazebo_ref prefix="right_foot_pitch" material="Gazebo/Blue"/>
-    <!--======================================================-->>
-    <!--======================================================-->>
-    <xacro:rot_link prefix="left_foot_pitch" rho="${rho_Fe}" r="${joint_cylinder_r}" l="${joint_cylinder_l}">
-        <xacro:rot_y_origin/>
-        <material name="blue"/>
-    </xacro:rot_link>
-    <xacro:default_rot_joint parent="left_foot_roll" child="left_foot_pitch">
-        <origin xyz="0 0 ${-2*joint_cylinder_r}"/>
-        <axis xyz="0 1 0"/>
-    </xacro:default_rot_joint>
-    <xacro:joint_trans parent="left_foot_roll" child="left_foot_pitch"/>
-    <xacro:gazebo_ref prefix="left_foot_pitch" material="Gazebo/Blue"/>
-    <!--======================================================-->>
-    <!--======================================================-->>
-    <xacro:cuboid_link prefix="right_foot" rho="${rho_Fe}" w="${foot_w}" d="${foot_d}" h="${foot_h}">
-        <material name="red"/>
-    </xacro:cuboid_link>
-    <xacro:default_fixed_joint parent="right_foot_pitch" child="right_foot">
-        <origin xyz="0 0 -${joint_cylinder_r+foot_h/2}"/>
-    </xacro:default_fixed_joint>
-    <xacro:gazebo_ref prefix="right_foot" material="Gazebo/Red"/>
-    <!--======================================================-->>
-    <!--======================================================-->>
-    <xacro:cuboid_link prefix="left_foot" rho="${rho_Fe}" w="${foot_w}" d="${foot_d}" h="${foot_h}">
-        <material name="red"/>
-    </xacro:cuboid_link>
-    <xacro:default_fixed_joint parent="left_foot_pitch" child="left_foot">
-        <origin xyz="0 0 -${joint_cylinder_r+foot_h/2}"/>
-    </xacro:default_fixed_joint>
-    <xacro:gazebo_ref prefix="left_foot" material="Gazebo/Red"/>
-    <!--======================================================-->>
+    <xacro:macro name="foot" params="name parent">
+        <xacro:solid_cylinder_link prefix="${name}_roll" rho="${rho_Fe}" r="${joint_cylinder_r}" l="${joint_cylinder_l}">
+            <xacro:rot_x_origin/>
+            <material name="yellow"/>
+        </xacro:solid_cylinder_link>
+        <xacro:rot_joint parent="${parent}" child="${name}_roll"
+                effort="${effort}" velocity="${velocity}" damping="${damping}">
+            <origin xyz="0 0 -${leg_lower_l/2+joint_cylinder_r}"/>
+            <axis xyz="1 0 0"/>
+        </xacro:rot_joint>
+        <xacro:effort_trans parent="${parent}" child="${name}_roll"/>
+        <xacro:gaz_link prefix="${name}_roll" material="Gazebo/Yellow" mu1="${mu1}" mu2="${mu2}"/>
+        <xacro:solid_cylinder_link prefix="${name}_pitch" rho="${rho_Fe}" r="${joint_cylinder_r}" l="${joint_cylinder_l}">
+            <xacro:rot_y_origin/>
+            <material name="blue"/>
+        </xacro:solid_cylinder_link>
+        <xacro:rot_joint parent="${name}_roll" child="${name}_pitch"
+                 effort="${effort}" velocity="${velocity}" damping="${damping}">
+            <origin xyz="0 0 ${-2*joint_cylinder_r}"/>
+            <axis xyz="0 1 0"/>
+        </xacro:rot_joint>
+        <xacro:effort_trans parent="${name}_roll" child="${name}_pitch"/>
+        <xacro:gaz_link prefix="${name}_pitch" material="Gazebo/Blue" mu1="${mu1}" mu2="${mu2}"/>
+        <xacro:solid_cuboid_link prefix="${name}" rho="${rho_Fe}" w="${foot_w}" d="${foot_d}" h="${foot_h}">
+            <material name="red"/>
+        </xacro:solid_cuboid_link>
+        <xacro:fixed_joint parent="${name}_pitch" child="${name}">
+            <origin xyz="0 0 -${joint_cylinder_r+foot_h/2}"/>
+        </xacro:fixed_joint>
+        <xacro:gaz_link prefix="${name}" material="Gazebo/Red" mu1="${mu1}" mu2="${mu2}"/>
+    </xacro:macro>
 </robot>

File: urdf/biped/lower_legs.urdf.xacro (robot description, xacro)
@@ -1,47 +1,24 @@
 <?xml version="1.0"?>
 <robot xmlns:xacro="http://www.ros.org/wiki/xacro">
-    <!--======================================================-->>
-    <xacro:rot_link prefix="right_lower_leg_roll" rho="${rho_Fe}" r="${joint_cylinder_r}" l="${joint_cylinder_l}">
-        <xacro:rot_x_origin/>
-        <material name="yellow"/>
-    </xacro:rot_link>
-    <xacro:default_rot_joint parent="right_upper_leg" child="right_lower_leg_roll">
-        <origin xyz="0 0 -${leg_upper_l/2+joint_cylinder_r}"/>
-        <axis xyz="1 0 0"/>
-    </xacro:default_rot_joint>
-    <xacro:joint_trans parent="right_upper_leg" child="right_lower_leg_roll"/>
-    <xacro:gazebo_ref prefix="right_lower_leg_roll" material="Gazebo/Yellow"/>
-    <!--======================================================-->>
-    <!--======================================================-->>
-    <xacro:rot_link prefix="left_lower_leg_roll" rho="${rho_Fe}" r="${joint_cylinder_r}" l="${joint_cylinder_l}">
-        <xacro:rot_x_origin/>
-        <material name="yellow"/>
-    </xacro:rot_link>
-    <xacro:default_rot_joint parent="left_upper_leg" child="left_lower_leg_roll">
-        <origin xyz="0 0 -${leg_upper_l/2+joint_cylinder_r}"/>
-        <axis xyz="1 0 0"/>
-    </xacro:default_rot_joint>
-    <xacro:joint_trans parent="left_upper_leg" child="left_lower_leg_roll"/>
-    <xacro:gazebo_ref prefix="left_lower_leg_roll" material="Gazebo/Yellow"/>
-    <!--======================================================-->>
-    <!--======================================================-->>
-    <xacro:rot_link prefix="right_lower_leg" rho="${rho_Fe}" r="${leg_lower_r}" l="${leg_lower_l}">
-        <origin xyz="0 0 0"/>
-        <material name="red"/>
-    </xacro:rot_link>
-    <xacro:default_fixed_joint parent="right_lower_leg_roll" child="right_lower_leg">
-        <origin xyz="0 0 -${joint_cylinder_r+leg_lower_l/2}"/>
-    </xacro:default_fixed_joint>
-    <xacro:gazebo_ref prefix="right_lower_leg" material="Gazebo/Red"/>
-    <!--======================================================-->>
-    <!--======================================================-->>
-    <xacro:rot_link prefix="left_lower_leg" rho="${rho_Fe}" r="${leg_lower_r}" l="${leg_lower_l}">
-        <origin xyz="0 0 0"/>
-        <material name="red"/>
-    </xacro:rot_link>
-    <xacro:default_fixed_joint parent="left_lower_leg_roll" child="left_lower_leg">
-        <origin xyz="0 0 -${joint_cylinder_r+leg_lower_l/2}"/>
-    </xacro:default_fixed_joint>
-    <xacro:gazebo_ref prefix="left_lower_leg" material="Gazebo/Red"/>
-    <!--======================================================-->>
+    <xacro:macro name="lower_leg" params="name parent">
+        <xacro:solid_cylinder_link prefix="${name}_roll" rho="${rho_Fe}" r="${joint_cylinder_r}" l="${joint_cylinder_l}">
+            <xacro:rot_x_origin/>
+            <material name="yellow"/>
+        </xacro:solid_cylinder_link>
+        <xacro:rot_joint parent="${parent}" child="${name}_roll"
+                effort="${effort}" velocity="${velocity}" damping="${damping}">
+            <origin xyz="0 0 -${leg_upper_l/2+joint_cylinder_r}"/>
+            <axis xyz="1 0 0"/>
+        </xacro:rot_joint>
+        <xacro:effort_trans parent="${parent}" child="${name}_roll"/>
+        <xacro:gaz_link prefix="${name}_roll" material="Gazebo/Yellow" mu1="${mu1}" mu2="${mu2}"/>
+        <xacro:solid_cylinder_link prefix="${name}" rho="${rho_Fe}" r="${leg_lower_r}" l="${leg_lower_l}">
+            <origin xyz="0 0 0"/>
+            <material name="red"/>
+        </xacro:solid_cylinder_link>
+        <xacro:fixed_joint parent="${name}_roll" child="${name}">
+            <origin xyz="0 0 -${joint_cylinder_r+leg_lower_l/2}"/>
+        </xacro:fixed_joint>
+        <xacro:gaz_link prefix="${name}" material="Gazebo/Red" mu1="${mu1}" mu2="${mu2}"/>
+    </xacro:macro>
 </robot>

File: urdf/biped/upper_legs.urdf.xacro (robot description, xacro)
@@ -1,71 +1,35 @@
 <?xml version="1.0"?>
 <robot xmlns:xacro="http://www.ros.org/wiki/xacro">
-    <!--======================================================-->>
-    <xacro:rot_link prefix="right_upper_leg_roll" rho="${rho_Fe}" r="${joint_cylinder_r}" l="${joint_cylinder_l}">
-        <xacro:rot_x_origin/>
-        <material name="yellow"/>
-    </xacro:rot_link>
-    <xacro:default_rot_joint parent="body" child="right_upper_leg_roll">
-        <origin xyz="${body_w/4} 0 -${body_h/2+joint_cylinder_r}"/>
-        <axis xyz="1 0 0"/>
-    </xacro:default_rot_joint>
-    <xacro:joint_trans parent="body" child="right_upper_leg_roll"/>
-    <xacro:gazebo_ref prefix="right_upper_leg_roll" material="Gazebo/Yellow"/>
-    <!--======================================================-->>
-    <!--======================================================-->>
-    <xacro:rot_link prefix="left_upper_leg_roll" rho="${rho_Fe}" r="${joint_cylinder_r}" l="${joint_cylinder_l}">
-        <xacro:rot_x_origin/>
-        <material name="yellow"/>
-    </xacro:rot_link>
-    <xacro:default_rot_joint parent="body" child="left_upper_leg_roll">
-        <origin xyz="${-body_w/4} 0 -${body_h/2+joint_cylinder_r}"/>
-        <axis xyz="1 0 0"/>
-    </xacro:default_rot_joint>
-    <xacro:joint_trans parent="body" child="left_upper_leg_roll"/>
-    <xacro:gazebo_ref prefix="left_upper_leg_roll" material="Gazebo/Yellow"/>
-    <!--======================================================-->>
-    <!--======================================================-->>
-    <xacro:rot_link prefix="right_upper_leg_pitch" rho="${rho_Fe}" r="${joint_cylinder_r}" l="${joint_cylinder_l}">
-        <xacro:rot_y_origin/>
-        <material name="blue"/>
-    </xacro:rot_link>
-    <xacro:default_rot_joint parent="right_upper_leg_roll" child="right_upper_leg_pitch">
-        <origin xyz="0 0 ${-2*joint_cylinder_r}"/>
-        <axis xyz="0 1 0"/>
-    </xacro:default_rot_joint>
-    <xacro:joint_trans parent="right_upper_leg_roll" child="right_upper_leg_pitch"/>
-    <xacro:gazebo_ref prefix="right_upper_leg_pitch" material="Gazebo/Blue"/>
-    <!--======================================================-->>
-    <!--======================================================-->>
-    <xacro:rot_link prefix="left_upper_leg_pitch" rho="${rho_Fe}" r="${joint_cylinder_r}" l="${joint_cylinder_l}">
-        <xacro:rot_y_origin/>
-        <material name="blue"/>
-    </xacro:rot_link>
-    <xacro:default_rot_joint parent="left_upper_leg_roll" child="left_upper_leg_pitch">
-        <origin xyz="0 0 ${-2*joint_cylinder_r}"/>
-        <axis xyz="0 1 0"/>
-    </xacro:default_rot_joint>
-    <xacro:joint_trans parent="left_upper_leg_roll" child="left_upper_leg_pitch"/>
-    <xacro:gazebo_ref prefix="left_upper_leg_pitch" material="Gazebo/Blue"/>
-    <!--======================================================-->>
-    <!--======================================================-->>
-    <xacro:rot_link prefix="right_upper_leg" rho="${rho_Fe}" r="${leg_upper_r}" l="${leg_upper_l}">
-        <origin xyz="0 0 0"/>
-        <material name="red"/>
-    </xacro:rot_link>
-    <xacro:default_fixed_joint parent="right_upper_leg_pitch" child="right_upper_leg">
-        <origin xyz="0 0 -${joint_cylinder_r+leg_upper_l/2}"/>
-    </xacro:default_fixed_joint>
-    <xacro:gazebo_ref prefix="right_upper_leg" material="Gazebo/Red"/>
-    <!--======================================================-->>
-    <!--======================================================-->>
-    <xacro:rot_link prefix="left_upper_leg" rho="${rho_Fe}" r="${leg_upper_r}" l="${leg_upper_l}">
-        <origin xyz="0 0 0"/>
-        <material name="red"/>
-    </xacro:rot_link>
-    <xacro:default_fixed_joint parent="left_upper_leg_pitch" child="left_upper_leg">
-        <origin xyz="0 0 -${joint_cylinder_r+leg_upper_l/2}"/>
-    </xacro:default_fixed_joint>
-    <xacro:gazebo_ref prefix="left_upper_leg" material="Gazebo/Red"/>
-    <!--======================================================-->>
+    <xacro:macro name="upper_leg" params="name parent reflect">
+        <xacro:solid_cylinder_link prefix="${name}_roll" rho="${rho_Fe}" r="${joint_cylinder_r}" l="${joint_cylinder_l}">
+            <xacro:rot_x_origin/>
+            <material name="yellow"/>
+        </xacro:solid_cylinder_link>
+        <xacro:rot_joint parent="${parent}" child="${name}_roll"
+                effort="${effort}" velocity="${velocity}" damping="${damping}">
+            <origin xyz="${reflect*body_w/4} 0 -${body_h/2+joint_cylinder_r}"/>
+            <axis xyz="1 0 0"/>
+        </xacro:rot_joint>
+        <xacro:effort_trans parent="${parent}" child="${name}_roll"/>
+        <xacro:gaz_link prefix="${name}_roll" material="Gazebo/Yellow" mu1="${mu1}" mu2="${mu2}"/>
+        <xacro:solid_cylinder_link prefix="${name}_pitch" rho="${rho_Fe}" r="${joint_cylinder_r}" l="${joint_cylinder_l}">
+            <xacro:rot_y_origin/>
+            <material name="blue"/>
+        </xacro:solid_cylinder_link>
+        <xacro:rot_joint parent="${name}_roll" child="${name}_pitch"
+                effort="${effort}" velocity="${velocity}" damping="${damping}">
+            <origin xyz="0 0 ${-2*joint_cylinder_r}"/>
+            <axis xyz="0 1 0"/>
+        </xacro:rot_joint>
+        <xacro:effort_trans parent="${name}_roll" child="${name}_pitch"/>
+        <xacro:gaz_link prefix="${name}_pitch" material="Gazebo/Blue" mu1="${mu1}" mu2="${mu2}"/>
+        <xacro:solid_cylinder_link prefix="${name}" rho="${rho_Fe}" r="${leg_upper_r}" l="${leg_upper_l}">
+            <origin xyz="0 0 0"/>
+            <material name="red"/>
+        </xacro:solid_cylinder_link>
+        <xacro:fixed_joint parent="${name}_pitch" child="${name}">
+            <origin xyz="0 0 -${joint_cylinder_r+leg_upper_l/2}"/>
+        </xacro:fixed_joint>
+        <xacro:gaz_link prefix="${name}" material="Gazebo/Red" mu1="${mu1}" mu2="${mu2}"/>
+    </xacro:macro>
 </robot>
